Commit message: Fixed merge conflict

File: robot/urdf/stretch_nobase_raised.urdf (robot description, URDF)
Before this commit: robot stretch_description, 38 links, 37 joints
Links:
- added link camera_accel_frame
- added link camera_accel_optical_frame
- added link camera_gyro_frame
- added link camera_gyro_optical_frame
- added link laser, mass 0.0749979022894495; collision mesh filename=package://stretch_description/meshes/laser.STL; visual mesh filename=package://stretch_description/meshes/laser.STL
- added link link_grasp_center
- added link link_left_wheel, mass 0.01; collision mesh filename=package://stretch_description/meshes/link_left_wheel.STL; visual mesh filename=package://stretch_description/meshes/link_left_wheel.STL
- added link link_right_wheel, mass 0.01; collision mesh filename=package://stretch_description/meshes/link_right_wheel.STL; visual mesh filename=package://stretch_description/meshes/link_right_wheel.STL
- link base_link: mass 1.07237826598 -> 1.0723782659782; geometry collision mesh filename=package://stretch_description/meshes/base_link.STL; visual mesh filename=package://stretch_description/meshes/base_link.STL
- link camera_link: mass 0.564 -> 0.072
- link link_arm_l0: mass 0.101241250325 -> 0.101241250325294
- link link_arm_l1: mass 0.0511763619538 -> 0.0511763619538321
- link link_arm_l2: mass 0.0569074368576 -> 0.0569074368576238
- link link_arm_l3: mass 0.0626921047058 -> 0.0626921047058405
- link link_arm_l4: mass 0.067652545579 -> 0.0676525455789735
- link link_aruco_inner_wrist: mass 0.000225 -> 0.0
- link link_aruco_left_base: mass 3.5999999999e-06 -> 3.59999999990368e-06
- link link_aruco_right_base: mass 3.5999999999e-06 -> 3.59999999990368e-06
- link link_aruco_shoulder: mass 0.000399141592654 -> 0.0
- link link_aruco_top_wrist: mass 0.000225 -> 0.0
- link link_gripper_finger_left: mass 0.0476207785199 -> 0.0476207785199479
- link link_gripper_fingertip_left: mass 0.00382160686585 -> 0.00382160686584851
- link link_gripper_fingertip_right: mass 0.00382160881469 -> 0.00382160881468841
- link link_head: mass 0.129454717596 -> 0.129454717596498
- link link_head_pan: mass 0.0358583411826 -> 0.035858341182617
- link link_head_tilt: mass 0.0701242408063 -> 0.0701242408063442
- link link_lift: mass 0.444820831236 -> 0.444820831236007
- link link_mast: mass 0.749143203376 -> 0.749143203376401
- link link_straight_gripper: mass 0.0496384234458 -> 0.0496384234458284
- link link_wrist_pitch: mass 0.0701267146296 -> 0.0701267146295583
- link link_wrist_roll: mass 0.00585666394359 -> 0.00585666394358811
- link link_wrist_yaw: mass 0.0405398981326 -> 0.0405398981326229
- link link_wrist_yaw_bottom: mass 0.09889068164 -> 0.0988906816399982
- link respeaker_base: mass 0.00969129410417 -> 0.00969129410417277
Joints:
- added joint camera_accel_joint: type fixed, parent camera_link, child camera_accel_frame, origin xyz=-0.01174 -0.00552 0.0051 rpy=0.0 0.0 0.0
- added joint camera_accel_optical_joint: type fixed, parent camera_accel_frame, child camera_accel_optical_frame, origin xyz=0.0 0.0 0.0 rpy=-1.5707963267948966 0.0 -1.5707963267948966
- added joint camera_gyro_joint: type fixed, parent camera_link, child camera_gyro_frame, origin xyz=-0.01174 -0.00552 0.0051 rpy=0.0 0.0 0.0
- added joint camera_gyro_optical_joint: type fixed, parent camera_gyro_frame, child camera_gyro_optical_frame, origin xyz=0.0 0.0 0.0 rpy=-1.5707963267948966 0.0 -1.5707963267948966
- added joint joint_grasp_center: type fixed, parent link_straight_gripper, child link_grasp_center, origin xyz=0.0 0.0 0.23 rpy=-1.5707963267949 -1.5707963267949 0.0
- added joint joint_laser: type fixed, parent base_link, child laser, origin xyz=0.000502800000000914 0.0 0.1664 rpy=0.0 0.0 -3.14159265358979, axis 0.0 0.0 0.0
- added joint joint_left_wheel: type continuous, parent base_link, child link_left_wheel, origin xyz=-0.00300000000001899 0.15765 0.0507999999999994 rpy=-1.5707963267949 3.16227047920818e-31 7.88745438253713e-16, axis 0.0 0.0 1.0
- added joint joint_right_wheel: type continuous, parent base_link, child link_right_wheel, origin xyz=-0.00300000000000034 -0.15765 0.0508000000000004 rpy=-1.57079632679489 -1.11022302462516e-16 7.28583859910277e-17, axis 0.0 0.0 1.0
- joint camera_color_optical_joint: origin xyz=0.0 0.0 0.0 rpy=-1.57079632679 0.0 -1.57079632679 -> xyz=0.0 0.0 0.0 rpy=-1.5707963267948966 0.0 -1.5707963267948966
- joint camera_depth_optical_joint: origin xyz=0.0 0.0 0.0 rpy=-1.57079632679 0.0 -1.57079632679 -> xyz=0.0 0.0 0.0 rpy=-1.5707963267948966 0.0 -1.5707963267948966
- joint camera_infra1_optical_joint: origin xyz=0.0 0.0 0.0 rpy=-1.57079632679 0.0 -1.57079632679 -> xyz=0.0 0.0 0.0 rpy=-1.5707963267948966 0.0 -1.5707963267948966
- joint camera_infra2_optical_joint: origin xyz=0.0 0.0 0.0 rpy=-1.57079632679 0.0 -1.57079632679 -> xyz=0.0 0.0 0.0 rpy=-1.5707963267948966 0.0 -1.5707963267948966
- joint camera_joint: origin xyz=0.027635246443941188 -0.007891582542698037 0.018816141866816533 rpy=0.023678437121446152 0.03004038358526162 0.02497239181338808 -> xyz=0.02523784681394068 -0.010728834303101144 0.01830933439884389 rpy=0.0034004333353294296 0.0075730565536364924 0.03847594366681832
- joint camera_link_joint: origin xyz=0.0106 0.0175 0.0125 rpy=0.0 0.0 0.0 -> xyz=0.010600000000000002 0.0175 0.0125 rpy=0.0 0.0 0.0
- joint joint_arm_l0: origin xyz=0.0 0.0 -0.01375 rpy=-3.05317390622e-16 -4.23236224077e-16 -2.68425135229e-17 -> xyz=0.0 0.0 -0.0137499999999938 rpy=-3.05317390622457e-16 -4.23236224076729e-16 -2.68425135229209e-17
- joint joint_arm_l1: origin xyz=0.0 0.0 0.013 rpy=7.41596560408e-17 1.33876788297e-16 -2.44545873596e-16 -> xyz=0.0 0.0 0.013 rpy=7.41596560408007e-17 1.33876788296791e-16 -2.44545873596083e-16
- joint joint_arm_l2: origin xyz=0.0 0.0 0.013 rpy=2.91385731014e-16 4.44300759505e-17 3.25691080516e-16 -> xyz=0.0 0.0 0.013 rpy=2.91385731014123e-16 4.44300759504684e-17 3.25691080516352e-16
- joint joint_arm_l4: origin xyz=-0.2523424694952765 -0.008046363015647639 0.0006448950170409711 rpy=1.5791021833517116 -0.015822158041521206 -1.5391794340439013 -> xyz=-0.26108831943305866 -0.002668423842320196 -0.0071486738136101475 rpy=1.5702311305669419 -0.049402943377846675 -1.593784844992891
- joint joint_aruco_inner_wrist: origin xyz=0.04725 -0.0119 -0.0272499999992 rpy=3.14159265359 4.23377442363e-14 3.14159265359 -> xyz=0.0472499999999947 -0.0119000000000034 -0.0272499999991938 rpy=3.14159265358979 4.23377442363088e-14 3.14159265358979
- joint joint_aruco_left_base: origin xyz=-0.005 0.1304972 0.1597482 rpy=0.0 0.0 -1.57079632679 -> xyz=-0.00500000000000014 0.1304972 0.1597482 rpy=0.0 0.0 -1.5707963267949
- joint joint_aruco_right_base: origin xyz=-0.005 -0.1304972 0.1597482 rpy=0.0 0.0 -1.57079632679 -> xyz=-0.00500000000000014 -0.1304972 0.1597482 rpy=0.0 0.0 -1.5707963267949
- joint joint_aruco_shoulder: origin xyz=-0.0133768876375 0.0558540528812 0.0861368272418 rpy=-1.53998860118e-29 3.55962409571e-15 0.0 -> xyz=-0.0133768876375287 0.0558540528812078 0.0861368272417975 rpy=-1.53998860117704e-29 3.55962409571165e-15 0.0
- joint joint_aruco_top_wrist: origin xyz=0.04725 0.029285 0.0 rpy=1.57079632679 -8.03728587323e-15 3.14159265359 -> xyz=0.0472500000000019 0.0292850000000015 0.0 rpy=1.5707963267949 -8.03728587323464e-15 3.14159265358979
- joint joint_gripper_fingertip_left: origin xyz=0.190596948564 -0.015 0.0 rpy=1.57079632679 4.51275387511e-14 2.60113659716 -> xyz=0.190596948563868 -0.015 0.0 rpy=1.57079632679496 4.51275387511463e-14 2.60113659715756
- joint joint_gripper_fingertip_right: origin xyz=-0.190596948564 -0.015 0.0 rpy=-1.57079632679 -3.43320051448e-14 0.540456056432 -> xyz=-0.190596948563868 -0.015 0.0 rpy=-1.57079632679483 -3.43320051448326e-14 0.540456056432235
- joint joint_head_pan: origin xyz=0.13352674158752487 0.07459624225825542 -0.011949505096590759 rpy=0.03234773727745851 0.03958515753515446 1.638065297966394 -> xyz=0.13722911390197282 0.07332566259307066 0.0023163937819581475 rpy=0.0007482311403641432 -0.007974668284138842 1.5877030998672819
- joint joint_head_tilt: origin xyz=-0.0031246655818673212 0.026367145294018252 -0.0541783861284751 rpy=1.5158113810665304 -0.04604807801866628 -0.008557149569685113 -> xyz=0.0061659563047586664 0.031097681644125918 -0.04811431501704618 rpy=1.5803818439877801 0.02649184343344646 -0.024781994225459944
- joint joint_lift: origin xyz=-0.0369217062323 0.1654712 -0.000341653286794 rpy=-1.5707963268 1.56154313753 -6.29420043665e-13 -> xyz=-0.0369217062323472 0.165471199999996 -0.000341653286793524 rpy=-1.57079632679552 1.5615431375292 -6.2942004366467e-13
- joint joint_mast: limit lower=0.0 upper=1.1 effort=100.0 velocity=1.0 -> (none); origin xyz=-0.07011542275174251 0.13318957636490408 0.026943480905560507 rpy=1.5898287663349295 -0.0009894011242959078 -0.003138498745985321 -> xyz=-0.07472892526522688 0.13537756859064354 0.03714847758175086 rpy=1.537328738240864 0.003131220662897949 0.011800923968804193
- joint joint_raised_gripper: origin xyz=0.03 -0.085 0.0355 rpy=3.14 0.261799 1.57 -> xyz=0.0 -0.09 0.047 rpy=3.14 0.261799 1.57
- joint joint_respeaker: origin xyz=1.09074743138e-05 1.36992 0.00303572796911 rpy=1.5707963268 0.0 3.14159265359 -> xyz=1.09074743137871e-05 1.36992 0.00303572796911382 rpy=1.57079632679553 0.0 3.14159265358916
- joint joint_straight_gripper: origin xyz=0.0 0.0 0.0155 rpy=3.54987407349e-30 3.24021254484e-20 -3.14159265359 -> xyz=0.0 0.0 0.0155 rpy=3.54987407349455e-30 3.24021254484265e-20 -3.14159265358979
- joint joint_wrist_pitch: origin xyz=0.0 -0.01955 -0.02475 rpy=1.57079632679 -8.12895570883e-15 -3.14159265359 -> xyz=0.0 -0.0195500000000002 -0.0247499999999984 rpy=1.5707963267949 -8.12895570882604e-15 -3.14159265358979
- joint joint_wrist_roll: origin xyz=-0.0188587444076 -0.0239999999999 0.01955 rpy=3.14159265359 1.57079632679 0.0 -> xyz=-0.0188587444076125 -0.0239999999998942 0.01955 rpy=3.14159265358979 1.5707963267949 0.0
- joint joint_wrist_yaw_bottom: origin xyz=0.0 0.0 0.0 rpy=-3.14159265359 1.13367999021e-14 1.57079632679 -> xyz=0.0 0.0 0.0 rpy=-3.14159265358979 1.13367999021379e-14 1.57079632679489
